Commit message: Updated robot model
Added wheels plugins

File: urdf/my_robot.xacro (robot description, xacro)
@@ -4,22 +4,4 @@
     <color rgba="0.0 0.0 0.0 1.0"/>
   </material>
-  <!-- <material name="blue">
-    <color rgba="0.203125 0.23828125 0.28515625 1.0"/>
-  </material>
-  <material name="green">
-    <color rgba="0.0 0.8 0.0 1.0"/>
-  </material>
-  <material name="grey">
-    <color rgba="0.2 0.2 0.2 1.0"/>
-  </material>
-  <material name="orange">
-    <color rgba="1.0 0.423529411765 0.0392156862745 1.0"/>
-  </material>
-  <material name="brown">
-    <color rgba="0.870588235294 0.811764705882 0.764705882353 1.0"/>
-  </material>
-  <material name="red">
-    <color rgba="0.80078125 0.12890625 0.1328125 1.0"/>
-  </material> -->
   <material name="white">
     <color rgba="1.0 1.0 1.0 1.0"/>
@@ -43,5 +25,5 @@
     <collision name="collision_chassis">
       <geometry>
-        <box size="0.4 0.2 0.07"/>
+        <box size="0.4 0.3 0.07"/>
       </geometry>
     </collision>
@@ -49,5 +31,5 @@
       <origin rpy="0 0 0" xyz="0 0 0"/>
       <geometry>
-        <box size="0.4 0.2 0.07"/>
+        <box size="0.4 0.3 0.07"/>
       </geometry>
       <material name="white"/>
@@ -55,7 +37,7 @@
     <!-- Castor Wheel -->
     <collision name="castor">
-      <origin rpy=" 0 0 0" xyz="0.25 0 -0.05"/>
+      <origin rpy=" 0 0 0" xyz="0.20 0 -0.05"/>
       <geometry>
-        <sphere radius="0.05"/>
+        <sphere radius="0.04"/>
       </geometry>
       <surface>
@@ -71,7 +53,7 @@
     </collision>
     <visual name="castor_visual">
-      <origin rpy=" 0 0 0" xyz="0.2 0 -0.05"/>
+      <origin rpy=" 0 0 0" xyz="0.15 0 -0.05"/>
       <geometry>
-        <sphere radius="0.05"/>
+        <sphere radius="0.04"/>
       </geometry>
     </visual>
@@ -87,5 +69,5 @@
       <origin rpy="0 1.5707 1.5707" xyz="0 0 0" />
       <geometry>
-        <cylinder length="0.04" radius="0.1"/>
+        <cylinder length="0.04" radius="0.08"/>
       </geometry>
     </collision>
@@ -93,6 +75,7 @@
       <origin rpy="0 1.5707 1.5707" xyz="0 0 0"/>
       <geometry>
-        <cylinder length="0.04" radius="0.1"/>
+        <cylinder length="0.04" radius="0.08"/>
       </geometry>
+      <material name="Black" />
     </visual>
   </link>
@@ -116,5 +99,5 @@
       <origin rpy="0 1.5707 1.5707" xyz="0 0 0" />
       <geometry>
-        <cylinder length="0.04" radius="0.1"/>
+        <cylinder length="0.04" radius="0.08"/>
       </geometry>
     </collision>
@@ -122,9 +105,10 @@
       <origin rpy="0 1.5707 1.5707" xyz="0 0 0"/>
       <geometry>
-        <cylinder length="0.04" radius="0.1"/>
+        <cylinder length="0.04" radius="0.08"/>
       </geometry>
+      <material name="Black" />
     </visual>
   </link>
-  <!-- Right Wheel Joint -->
+  <!-- Left Wheel Joint -->
   <joint name="joint_left_wheel" type="continuous">
     <origin rpy="0 0 0" xyz="-0.05 -0.15 0"/>
@@ -135,3 +119,20 @@
     <joint_properties damping="1.0" friction="1.0" />
   </joint>
+  <!-- Plugins -->
+  <gazebo>
+    <plugin filename="libgazebo_ros_diff_drive.so" name="differential_drive_controller">
+      <alwaysOn>true</alwaysOn>
+      <legacyMode>false</legacyMode>
+      <updateRate>20</updateRate>
+      <leftJoint>joint_left_wheel</leftJoint>
+      <rightJoint>joint_right_wheel</rightJoint>
+      <wheelSeparation>0.4</wheelSeparation>
+      <wheelDiameter>0.2</wheelDiameter>
+      <torque>0.1</torque>
+      <commandTopic>cmd_vel</commandTopic>
+      <odometryTopic>odom</odometryTopic>
+      <odometryFrame>odom</odometryFrame>
+      <robotBaseFrame>link_chassis</robotBaseFrame>
+    </plugin>
+  </gazebo>
 </robot>

Commit message: Updated files

File: urdf/my_robot.xacro (robot description, xacro)
@@ -1,4 +1,5 @@
 <?xml version="1.0" ?>
 <robot name="my_robot">
+  <!-- Colors-->
   <material name="black">
     <color rgba="0.0 0.0 0.0 1.0"/>
@@ -7,4 +8,7 @@
     <color rgba="1.0 1.0 1.0 1.0"/>
   </material>
+  <material name = "red">
+    <color rgba = "1.0 0.0 0.0 1.0"/>
+  </material>
   <gazebo reference="link_chassis">
     <material>Gazebo/White</material>
@@ -39,5 +43,5 @@
       <origin rpy=" 0 0 0" xyz="0.20 0 -0.05"/>
       <geometry>
-        <sphere radius="0.04"/>
+        <sphere radius="0.03"/>
       </geometry>
       <surface>
@@ -55,5 +59,5 @@
       <origin rpy=" 0 0 0" xyz="0.15 0 -0.05"/>
       <geometry>
-        <sphere radius="0.04"/>
+        <sphere radius="0.03"/>
       </geometry>
     </visual>
@@ -136,3 +140,68 @@
     </plugin>
   </gazebo>
+  <!-- Laser Scanner -->
+   <link name="sensor_laser">
+    <inertial>
+      <origin xyz="0 0 0" rpy="0 0 0" />
+      <mass value="1" />
+      <!-- RANDOM INERTIA BELOW -->
+      <inertia ixx="0.02" ixy="0" ixz="0" iyy="0.02" iyz="0" izz="0.02"/>
+    </inertial>
+    <visual>
+      <origin xyz="0 0 0" rpy="0 0 0" />
+      <geometry>
+        <cylinder radius="0.05" length="0.1"/>
+      </geometry>
+      <material name="red" />
+    </visual>
+    <collision>
+      <origin xyz="0 0 0" rpy="0 0 0"/>
+      <geometry>
+        <cylinder radius="0.05" length="0.1"/>
+      </geometry>
+    </collision>
+  </link>
+  <joint name="joint_sensor_laser" type="fixed">
+    <origin xyz="0.15 0 0.05" rpy="0 0 0"/>
+    <parent link="link_chassis"/>
+    <child link="sensor_laser"/>
+  </joint>
+  <!-- Macro for Laser scanner-->
+  <xacro:macro name="cylinder_inertia" params="mass r l">
+    <inertia ixx="${mass*(3*r*r+l*l)/12}" ixy = "0" ixz = "0"
+                iyy="${mass*(3*r*r+l*l)/12}" iyz = "0" izz="${mass*(r*r)/2}" />
+  </xacro:macro>
+  <xacro:cylinder_inertia mass="1" r="0.05" l="0.1" />
+  <!--Laser Scanner plugin-->
+  <gazebo reference="sensor_laser">
+    <sensor type="ray" name="head_hokuyo_sensor">
+      <pose>0 0 0 0 0 0</pose>
+      <visualize>false</visualize>
+      <update_rate>20</update_rate>
+      <ray>
+        <scan>
+          <horizontal>
+            <samples>720</samples>
+            <resolution>1</resolution>
+            <min_angle>-1.570796</min_angle>
+            <max_angle>1.570796</max_angle>
+          </horizontal>
+        </scan>
+        <range>
+          <min>0.10</min>
+          <max>10.0</max>
+          <resolution>0.01</resolution>
+        </range>
+        <noise>
+          <type>gaussian</type>
+          <mean>0.0</mean>
+          <stddev>0.01</stddev>
+        </noise>
+      </ray>
+      <plugin name="gazebo_ros_head_hokuyo_controller" filename="libgazebo_ros_laser.so">
+        <topicName>/laser/scan</topicName>
+        <frameName>sensor_laser</frameName>
+      </plugin>
+    </sensor>
+  </gazebo>
 </robot>

Commit message: Updated and added ded files

File: urdf/my_robot.xacro (robot description, xacro)
@@ -14,9 +14,12 @@
     <material>Gazebo/White</material>
   </gazebo>
-  <gazebo reference="link_left_wheel">
+  <gazebo reference="left_wheel">
     <material>Gazebo/Black</material>
   </gazebo>
-  <gazebo reference="link_right_wheel">
+  <gazebo reference="right_wheel">
     <material>Gazebo/Black</material>
+  </gazebo>
+  <gazebo reference="sensor_laser">
+    <material>Gazebo/Red</material>
   </gazebo>
   <link name="link_chassis">
@@ -29,5 +32,5 @@
     <collision name="collision_chassis">
       <geometry>
-        <box size="0.4 0.3 0.07"/>
+        <box size="0.5 0.3 0.07"/>
       </geometry>
     </collision>
@@ -35,5 +38,5 @@
       <origin rpy="0 0 0" xyz="0 0 0"/>
       <geometry>
-        <box size="0.4 0.3 0.07"/>
+        <box size="0.5 0.3 0.07"/>
       </geometry>
       <material name="white"/>
@@ -41,7 +44,7 @@
     <!-- Castor Wheel -->
     <collision name="castor">
-      <origin rpy=" 0 0 0" xyz="0.20 0 -0.05"/>
-      <geometry>
-        <sphere radius="0.03"/>
+      <origin rpy=" 0 0 0" xyz="0.35 0 -0.05"/>
+      <geometry>
+        <sphere radius="0.05"/>
       </geometry>
       <surface>
@@ -57,7 +60,7 @@
     </collision>
     <visual name="castor_visual">
-      <origin rpy=" 0 0 0" xyz="0.15 0 -0.05"/>
-      <geometry>
-        <sphere radius="0.03"/>
+      <origin rpy=" 0 0 0" xyz="0.2 0 -0.05"/>
+      <geometry>
+        <sphere radius="0.05"/>
       </geometry>
     </visual>
@@ -73,5 +76,5 @@
       <origin rpy="0 1.5707 1.5707" xyz="0 0 0" />
       <geometry>
-        <cylinder length="0.04" radius="0.08"/>
+        <cylinder length="0.04" radius="0.1"/>
       </geometry>
     </collision>
@@ -79,5 +82,5 @@
       <origin rpy="0 1.5707 1.5707" xyz="0 0 0"/>
       <geometry>
-        <cylinder length="0.04" radius="0.08"/>
+        <cylinder length="0.04" radius="0.1"/>
       </geometry>
       <material name="Black" />
@@ -103,5 +106,5 @@
       <origin rpy="0 1.5707 1.5707" xyz="0 0 0" />
       <geometry>
-        <cylinder length="0.04" radius="0.08"/>
+        <cylinder length="0.04" radius="0.1"/>
       </geometry>
     </collision>
@@ -109,5 +112,5 @@
       <origin rpy="0 1.5707 1.5707" xyz="0 0 0"/>
       <geometry>
-        <cylinder length="0.04" radius="0.08"/>
+        <cylinder length="0.04" radius="0.1"/>
       </geometry>
       <material name="Black" />
